File: LED/LED Cube/LedCube_595_2x2891/LED_CUBE_595.brd (EAGLE design)
At the start: 99.4 x 30.5 mm, 37 parts, among them IC1 74LS595N, IC2 74LS595N, IC3 74LS595N, IC4 UDN2981A, IC5 UDN2981A, Q1 BSS84, Q2 BSS84, Q3 BSS84, Q4 BSS84, Q5 BSS84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

Commit message: added pin connection
Routing:
- net N$1: track 3.96 -> 5.87 mm
- net N$30: vias 2 -> 3
Changed lines of the file:
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@@
 <via x="2.54" y="22.86" extent="1-16" drill="0.8" diameter="1.6764"/>
 <wire x1="4.445" y1="24.765" x2="2.54" y2="22.86" width="0.6096" layer="16"/>
-<wire x1="5.715" y1="24.765" x2="38.735" y2="12.065" width="0" layer="19" extent="1-1"/>
+<wire x1="38.735" y1="12.065" x2="36.83" y2="12.065" width="0.4064" layer="16"/>
+<wire x1="36.83" y1="12.065" x2="5.715" y2="24.765" width="0" layer="19" extent="1-16"/>
 </signal>
 <signal name="N$2">
@@
 <wire x1="38.735" y1="24.765" x2="34.925" y2="24.765" width="0.4064" layer="16"/>
 <wire x1="38.735" y1="24.765" x2="69.85" y2="12.065" width="0" layer="19" extent="16-16"/>
+<via x="36.83" y="12.065" extent="1-16" drill="0.8" diameter="1.778"/>
 </signal>
 <signal name="N$32">
